Commit message: R2|车体传感器坐标复测定案（08-24）：base_link 离地 12cm、VLP-16 0.655m、G354 实测
- 改动: r2.urdf velodyne_joint z 0.56→0.655；sensor-mount 引用处同步（w1-operation/minimal-loop README/r2_sensors README）
- 原因: 08-24 实车复测（VLP-16 与 G354 安装微调后定案）：光学中心距地 77~78cm、base_link 离地 12cm（原 13）、G354 距地 30~31cm；高差 47cm 与 FAST-LIO 外参自洽
- 影响/注意: TF 树雷达高度修正 8cm（影响 Nav2 障碍物高度判断）；z_min 0.3 地面滤波阈值待下次建图验证是否同步上调（下射环抬高 ~0.1m）；retrospect 历史记录保留旧值

File: r2_sensors/config/r2.urdf (robot description, URDF)
Before this commit: robot r2, 2 links, 1 joints
Joints:
- joint velodyne_joint: origin xyz=0 0 0.56 -> xyz=0 0 0.655
